File: TSAL_plausibility.kicad_sch (KiCad schematic)
At the start: 32 parts, among them Q1 NMOS, U10 SN74HCS266PWR, U12 74LVC1G32GV, U14 OPA355NA, U3 74LVC2G74, U6 CD74HC30PWR, U7 4072, U8 4001, U9 74LVC1G32GV

Commit message: Added TSAC Indicator with PSU
Parts:
- C13: footprint Capacitor_SMD:CP_Elec_8x5.4 -> Capacitor_SMD:C_0603_1608Metric
Changed lines of the file:
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@@
 			)
 		)
-		(property "Footprint" "Capacitor_SMD:CP_Elec_8x5.4"
+		(property "Footprint" "Capacitor_SMD:C_0603_1608Metric"
 			(at 49.2252 176.53 0)
 			(effects
@@
 			)
 		)
+		(property "resistor datasheet" ""
+			(at 48.26 172.72 0)
+			(effects
+				(font
+					(size 1.27 1.27)
+				)
+			)
+		)
