File: TS_sense.kicad_sch (KiCad schematic)
At the start: 43 parts, among them J16 Conn_01x02, Q8 NMOS, U1 TPS7A0508PDBV, U11 OPA355NA, U13 SFH617A-1X007T, U16 TPS7A0508PDBV, U17 5245-AM50W-45024SNZ-ND, U22 TBA1-0511E, U24 SFH617A-1X007T, U25 OPA355NA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

Commit message: ordered
Parts:
- removed C16, C7: 0.47uF, Capacitor_SMD:C_0603_1608Metric, symbol Device:C
- removed C17, C6: 10uF, Capacitor_SMD:C_0603_1608Metric, symbol Device:C_Polarized
- removed C18, C20, C29, C5: 100nF, Capacitor_SMD:C_0603_1608Metric, symbol Device:C
- removed C19, C2: 1uF, Capacitor_SMD:C_0603_1608Metric, symbol Device:C
- removed C35: 100nF, Capacitor_SMD:C_0603_1608Metric, symbol Device:C_Small
- removed J16: Conn_01x02, wuerth_conn:66200211024, symbol Connector_Generic:Conn_01x02
- removed Q8: NMOS, Package_TO_SOT_SMD:SOT-23-3, symbol Simulation_SPICE:NMOS
- removed R32: 200R, symbol Device:R
- removed R33, R39: 1k, Resistor_SMD:R_0603_1608Metric, symbol Device:R
- removed R34: 12k, Resistor_SMD:R_0603_1608Metric, symbol Device:R
- removed R5: 10k, Resistor_SMD:R_0603_1608Metric, symbol Device:R
- removed U1, U16: TPS7A0508PDBV, Package_TO_SOT_SMD:SOT-23-5, symbol Regulator_Linear:TPS7A0508PDBV
- removed U17: 5245-AM50W-45024SNZ-ND, Converter_DCDC:Converter_DCDC_Murata_CRE1xxxxxxDC_THT, symbol Regulator_Switching:CRE1S0505DC
- removed U24: SFH617A-1X007T, Package_DIP:SMDIP-4_W9.53mm_Clearance8mm, symbol Isolator:SFH617A-1X007T
- removed U25: OPA355NA, Package_TO_SOT_SMD:SOT-23-6, symbol Amplifier_Operational:OPA355NA
- removed U5: PDS1-S24-S24-D, Converter_DCDC:Converter_DCDC_TRACO_TBA1-xxxxE_Single_THT, symbol Converter_DCDC:TBA1-0511E
Other:
- note removed: "Accumulator Indicator LED"
- note removed: "Footprint Issues"
