File: lv_connectors.kicad_sch (KiCad schematic)
At the start: 41 parts, among them J10 Conn_01x10, J11 Conn_01x04, J12 Conn_01x04, J14 Conn_01x04, J15 Conn_01x10, J2 Conn_01x04, J3 Conn_01x04, J4 Conn_01x04, J5 Conn_01x02, J6 Conn_01x02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

Commit message: ordered
Connections:
- net AIR1_SW: now also U18.9 (CH8); no longer U18.11 (CH6)
- net PRCH_SW: now also U18.11 (CH6); no longer U18.9 (CH8)
Changed lines of the file:
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@@
+		)
+	)
+	(hierarchical_label "PRCH_SW"
+		(shape output)
+		(at 123.19 39.37 0)
+		(fields_autoplaced yes)
+		(effects
+			(font
+				(size 1.27 1.27)
+			)
+			(justify left)
 		)
 	)
@@
 		(shape input)
 		(at 123.19 29.21 0)
+		(fields_autoplaced yes)
+		(effects
+			(font
+				(size 1.27 1.27)
+			)
+			(justify left)
+		)
+	)
+	(hierarchical_label "AIR1_SW"
+		(shape output)
+		(at 123.19 44.45 0)
 		(fields_autoplaced yes)
 		(effects
@@
 		(fields_autoplaced yes)
 		(effects
-			(font
-				(size 1.27 1.27)
-			)
-			(justify left)
-		)
-	)
-	(hierarchical_label "AIR1_SW"
-		(shape output)
-		(at 123.19 39.37 0)
-		(fields_autoplaced yes)
-		(effects
-			(font
-				(size 1.27 1.27)
-			)
-			(justify left)
-		)
-	)
-	(hierarchical_label "PRCH_SW"
-		(shape output)
-		(at 123.19 44.45 0)
-		(fields_autoplaced yes)
-		(effects
