File: rpm_TSAL_RED/rpm_TSAL_RED.kicad_sch (KiCad schematic)
At the start: 43 parts, among them J1 Conn_01x04, J2 Conn_01x04, J3 Conn_01x02, J4 Conn_01x01, J5 Conn_01x01, J6 Conn_01x02, Q1 NMOS, Q2 PMOS, U1 NE555D, U2 TBA1-0511E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

Commit message: Added Sub project
Connections:
- net TS+ is gone; now on net HV_RED+: R16.1
- net TS- is gone; now on net HV_RED-: C6.2, C7.2, C8.2, R10.1, R7.1, R9.1, U2.4 (-Vout), U4.2 (V-)
- net +24V: now also J1.1 (Pin_1)
- net +5V: now also J1.3 (Pin_3)
- net GND: now also J1.4 (Pin_4)
- net TSAL_RED_LED_SW: now also J1.2 (Pin_2)
Other:
- title: (none) -> RED TSAL Control
- moved on the sheet: J1, J2
